File: hardware/rev0A/pcb/rev0A.kicad_sch (KiCad schematic)
At the start: 63 parts, among them J1 TYPE-C-31-M-12, J2 Conn_01x02_Socket, J3 Conn_01x02_Socket, J4 Conn_01x02_Socket, J5 Conn_01x03_Socket, J6 Conn_01x02_Socket, J7 Conn_01x03_Socket, K1 SRD-05VDC-SL-C, K2 SRD-05VDC-SL-C, K3 SRD-05VDC-SL-C, Q1 BC337, Q2 BC337, Q3 BC337, SW1 SW_Push_Dual, SW2 SW_Push_Dual, U1 AMS1117, U2 LM2575-5.0BT, U3 ESP32-S3-WROOM-1, U4 TXS0102DCU, U5 ADC088S022CIMTX_NOPB

Commit message: PCB Progress
Parts:
- removed C3: 10uF, symbol Device:C
- removed C4, C9: 0.1uF, symbol Device:C
- removed D1: LED, symbol Device:LED
- removed D10: WS2812B-2020, LED_SMD:LED_WS2812B-2020_PLCC4_2.0x2.0mm, symbol LED:WS2812B-2020
- removed D2: 1N5824, symbol Device:D_Schottky
- removed D6: LESD5D5.0CT1G, LESD5D5.0CT1G:TVS_LESD5D5.0CT1G, symbol Drip:LESD5D5.0CT1G
- removed D9: 1N4148W, Diode_SMD:D_SOD-123, symbol Diode:1N4148W
- removed J4: Conn_01x02_Socket, symbol Connector:Conn_01x02_Socket
- removed J5: Conn_01x03_Socket, symbol Connector:Conn_01x03_Socket
- removed R1: 100, symbol Device:R
- removed R3: 5100, symbol Device:R
- removed R5, R7: 15000, symbol Device:R
- removed SW1, SW2: SW_Push_Dual, symbol Switch:SW_Push_Dual
- removed U3: ESP32-S3-WROOM-1, RF_Module:ESP32-S3-WROOM-1, symbol RF_Module:ESP32-S3-WROOM-1
- added C1: 100uF, easyeda2kicad:CAP-SMD_BD8.0-L8.3-W8.3-FD, symbol Device:C_Polarized
- added C14: 10uF, easyeda2kicad:C0805, symbol Device:C
- added C19, C20, C21, C22: 0.1uF, easyeda2kicad:C0402, symbol Device:C
- added C2: 330uF, easyeda2kicad:CAP-SMD_BD10.0-L10.3-W10.3-FD, symbol Device:C_Polarized
- added D1: 1N5822, easyeda2kicad:DO-201AD_BD5.3-L8.4-P12.50-D1.4-FD, symbol Diode:1N5822
- added D4: LESD5D5.0CT1G, easyeda2kicad:SOD-523_L1.2-W0.8-LS1.6-BI, symbol Drip:LESD5D5.0CT1G
- added D7: 1N4148W, easyeda2kicad:SOD-123_L2.8-W1.8-LS3.7-RD, symbol Diode:1N4148W
- added DC1: EJ508A, easyeda2kicad:DC-IN-TH_EJ508A, symbol easyeda2kicad:EJ508A
- added GPIO20, GPIO21, TP1, TP2: ~, TestPoint:TestPoint_Pad_2.0x2.0mm, symbol Connector:TestPoint
- added IC1: ESP32-C3-WROOM-02-H4, RF_Module:ESP32-C3-WROOM-02, symbol RF_Module:ESP32-C3-WROOM-02
- added J1: Conn_01x02_Socket, easyeda2kicad:CONN-TH_B2B-XH-A-LF-SN, symbol Connector:Conn_01x02_Socket
- added J4: Conn_01x03_Socket, easyeda2kicad:CONN-TH_3P-P2.50_A2501WV2-3P, symbol Connector:Conn_01x03_Socket
- added J7: Conn_01x06_Socket, easyeda2kicad:HDR-TH_6P-P2.54-V-F, symbol Connector:Conn_01x06_Socket
- added LED1: WS2812B-2020, easyeda2kicad:LED-SMD_4P-L2.0-W2.0-TL_WS2812B-2020, symbol easyeda2kicad:WS2812B-2020
- added R11: 1000, easyeda2kicad:R0603, symbol Device:R
- added R2: 10000, easyeda2kicad:R1206, symbol Device:R
- added R4: 5100, easyeda2kicad:R0603, symbol Device:R
- added SW1, SW2: SW_Push, easyeda2kicad:SW-TH_5P-L6.0-W6.0-P4.50-LS6.5, symbol Switch:SW_Push
- added TP10, TP11, TP12, TP13, TP3, TP4, TP5, TP6, TP7, TP8, TP9: TestPoint, TestPoint:TestPoint_Pad_2.0x2.0mm, symbol Connector:TestPoint
- C10: value 10uF -> 22pF; footprint (none) -> easyeda2kicad:C0603; LCSC Part (none) -> C1653
- C11: value 0.1uF -> 22pF; footprint (none) -> easyeda2kicad:C0603; LCSC Part (none) -> C1653
- C12, C13: value 1nF -> 0.1uF; footprint (none) -> easyeda2kicad:C0402; LCSC Part (none) -> C1525
- C15: value 0.1uF -> 10uF; footprint (none) -> easyeda2kicad:C0805; LCSC Part (none) -> C1713
- C16, C18: footprint (none) -> easyeda2kicad:C0402; LCSC Part (none) -> C1525
- C17, C7: footprint (none) -> easyeda2kicad:C0805; LCSC Part (none) -> C1713
- C3: renamed from C1; footprint (none) -> easyeda2kicad:C0805; LCSC Part (none) -> C1713
- C4: renamed from C2; footprint (none) -> easyeda2kicad:C0402; LCSC Part (none) -> C1525
- C5: value 680uF -> 10uF; footprint (none) -> easyeda2kicad:C0805; LCSC Part (none) -> C1713
- C6: value 220uF -> 0.1uF; footprint (none) -> easyeda2kicad:C0402; LCSC Part (none) -> C1525
- C8: value 10uF -> 0.1uF; footprint (none) -> easyeda2kicad:C0402; LCSC Part (none) -> C1525
- C9: renamed from C14; footprint (none) -> easyeda2kicad:C0603; LCSC Part (none) -> C1592
- D2: renamed from D3; footprint Diode_THT:D_DO-41_SOD81_P10.16mm_Horizontal -> easyeda2kicad:SOD-123_L2.7-W1.6-LS3.7-RD; LCSC Part (none) -> C82544
- D3: renamed from D4; footprint LESD5D5.0CT1G:TVS_LESD5D5.0CT1G -> easyeda2kicad:SOD-523_L1.2-W0.8-LS1.6-BI; LCSC Part (none) -> C383211
- D5: footprint LESD5D5.0CT1G:TVS_LESD5D5.0CT1G -> easyeda2kicad:SOD-523_L1.2-W0.8-LS1.6-BI; LCSC Part (none) -> C383211
- D6: renamed from D7; footprint Diode_SMD:D_SOD-123 -> easyeda2kicad:SOD-123_L2.8-W1.8-LS3.7-RD; LCSC Part (none) -> C2099
- D8: footprint Diode_SMD:D_SOD-123 -> easyeda2kicad:SOD-123_L2.8-W1.8-LS3.7-RD; LCSC Part (none) -> C2099
- IC2: renamed from U4; LCSC Part (none) -> C53434
- IC3: renamed from U5; footprint ADC088S022CIMTX_NOPB:SOP65P640X120-16N -> easyeda2kicad:TSSOP-16_L5.0-W4.4-P0.65-LS6.4-BL; LCSC Part (none) -> C701585
- J2, J3: footprint (none) -> easyeda2kicad:CONN-TH_B2B-XH-A-LF-SN; LCSC Part (none) -> C158012
- J5: renamed from J6; footprint (none) -> easyeda2kicad:CONN-TH_B2B-XH-A-LF-SN; LCSC Part (none) -> C158012
- J6: renamed from J7; footprint (none) -> easyeda2kicad:CONN-TH_3P-P2.50_A2501WV2-3P; LCSC Part (none) -> C144394
- K1, K2, K3: value SRD-05VDC-SL-C -> SRD-12VDC-SL-C; footprint SRD-05VDC-SL-C:RELAY_SRD-05VDC-SL-C -> easyeda2kicad:RELAY-TH_SRD-XXVDC-XL-C; LCSC Part (none) -> C30431
- L1: value 33uH -> 330uH; footprint (none) -> easyeda2kicad:IND-SMD_L12.3-W12.3; LCSC Part (none) -> 10152
- Q1, Q2, Q3: footprint Package_TO_SOT_THT:TO-92_Inline -> easyeda2kicad:TO-92-3_L4.8-W3.7-P2.54-R; LCSC Part (none) -> C328602
- R1: renamed from R14; footprint (none) -> easyeda2kicad:R1206; LCSC Part (none) -> C1489
- R10: footprint (none) -> easyeda2kicad:R1206; LCSC Part (none) -> C1489
- R12, R13: value R -> 10000; footprint (none) -> easyeda2kicad:R1206; LCSC Part (none) -> C1489
- R3: renamed from R2; footprint (none) -> easyeda2kicad:R0603; LCSC Part (none) -> C23186
- R5: renamed from R11; value 250 -> 220; footprint (none) -> easyeda2kicad:RES-TH_BD2.3-L6.5-P10.50-D0.5; LCSC Part (none) -> C714546
- R6, R8: value 2700 -> 10000; footprint (none) -> easyeda2kicad:R1206; LCSC Part (none) -> C1489
- R7: renamed from R4; value 2700 -> 1000; footprint (none) -> easyeda2kicad:R0603; LCSC Part (none) -> C21190
- R9: value 15000 -> 1000; footprint (none) -> easyeda2kicad:R0603; LCSC Part (none) -> C21190
- USBC1: renamed from J1; footprint (none) -> easyeda2kicad:USB-C_SMD-TYPE-C-31-M-12; LCSC Part (none) -> C165948
- VREG1: renamed from U2; value LM2575-5.0BT -> LM2575T-5.0; footprint Package_TO_SOT_THT:TO-220-5_Vertical -> easyeda2kicad:TO-263-5_L10.2-W8.9-P1.70-TL; LCSC Part (none) -> C12061
- VREG2: renamed from U1; LCSC Part (none) -> C6186
Connections:
- net GPIO0 is gone; now on net GND: C15.1, R12.2
- net +12V: now also D6.1 (K), D8.1 (K), K1.C1, K1.COM, K2.C1, K2.COM, K3.C1, K3.COM, C1.1, D7.1 (K), DC1.1, TP2.1; no longer C5.1, J2.1 (Pin_1), J3.1 (Pin_1), K1.NO, K2.NO, K3.NO
- net +3.3V: now also C17.1, C18.1, C5.1, C6.1, C21.2, LED1.4 (VDD), TP4.1; no longer C8.1
- net +3V3: now also C7.2, C8.2, IC1.1 (3V3), J7.3 (Pin_3), R2.1; no longer C17.1, C18.1, R12.1, R13.1
- net +5V: now also C15.2, C16.2, C14.1, C2.1, C22.1, J4.1 (Pin_1), TP3.1, TP8.1; no longer C10.1, C11.1, C6.1, C7.1, D6.1 (K), D8.1 (K), K1.A1, K2.A1, K3.A1
- net ACD Chip Select: now also IC1.15 (IO3)
- net ACD Program: now also IC1.18 (IO0)
- net CHIP_PU: now also C13.1, IC1.2 (EN), J7.2 (Pin_2), SW2.3, SW2.4, TP5.1; no longer C16.1, R13.2
- net D+: now also C10.1, D5.2, IC1.14 (IO19), TP6.1
- net D-: now also C11.1, D4.2, IC1.13 (IO18), TP7.1; no longer D5.2
- net Flow Sensor Data: now also IC1.10 (IO10), TP11.1
- net Flow Sensor Enable: now also R6.2, IC1.7 (IO8); no longer R10.2
- net GND: now also C16.1, C7.1, C8.1, R10.2, R6.1, R8.2, USBC1.A1 (GND), USBC1.A12 (GND), USBC1.B1 (GND), USBC1.B12 (GND), VREG1.6 (TAB(GND)), C1.2, C14.2, C19.2, C2.2, C20.2, C21.1, C22.2, D1.2 (A), D4.1, DC1.2, IC1.19 (GND), IC1.9 (GND), J1.2 (Pin_2), J4.3 (Pin_3), J7.6 (Pin_6), LED1.2 (GND), R4.2, SW1.1, SW1.2, SW2.1, SW2.2, TP1.1; no longer C15.2, C16.2, C7.2, C8.2, K1.COM, K2.COM, K3.COM, R10.1, R9.1, USBC1.A1_B12 (GND), USBC1.B1_A12 (GND)
- net Pressure Sensor (Current): now also R13.1, C20.1, TP9.1; no longer C12.1, J5.2 (Pin_2), R5.1
- net Pressure Sensor (Voltage): now also C19.1, TP10.1; no longer C13.1
- net RGB: now also IC1.3 (IO4), LED1.3 (DI)
- net Relay1: now also IC1.4 (IO5)
- net Relay2: now also R9.1, IC1.5 (IO6); no longer R6.1
- net Relay3: now also IC1.6 (IO7), R11.1; no longer R8.1
- net SCLK: now also IC1.17 (IO1)
- net SDA: now also IC1.16 (IO2)
- net at Q3.1 (C): now also D8.2 (A), K3.C2; no longer K3.A2
- net at D2.2 (A), D3.2: now also USBC1.A4 (VBUS), USBC1.A9 (VBUS), USBC1.B4 (VBUS), USBC1.B9 (VBUS); no longer USBC1.A4_B9 (VBUS), USBC1.B4_A9 (VBUS)
- net at USBC1.B5 (CC2): now also R4.1
- net at L1.1, VREG1.2 (OUT): now also D1.1 (K)
- net at Q1.2 (B), R7.2: now also R8.1
- net at D6.2 (A), Q1.1 (C): now also K1.C2; no longer K1.A2
- net at Q2.2 (B): now also R10.1, R9.2; no longer R6.2
- net at IC2.1 (B2): now also TP13.1
- net at IC2.4 (A2): now also TP12.1
- net at IC2.8 (B1): now also J4.2 (Pin_2)
- new net: J5.2 (Pin_2), R13.2, R5.1
- new net: J3.1 (Pin_1), K3.NO
- new net: Q3.2 (B), R11.2, R12.1
- new net: D7.2 (A), K2.C2, Q2.1 (C)
- new net: J2.1 (Pin_1), K2.NO
- new net: J1.1 (Pin_1), K1.NO
- new net GPIO9: C12.1, IC1.8 (IO9), J7.1 (Pin_1), R2.2, SW1.3, SW1.4
- new net IO20: IC1.11 (IO20/RXD), J7.5 (Pin_5)
- new net IO21: IC1.12 (IO21/TXD), J7.4 (Pin_4)
- no-connect marks 8 -> 7
Other:
- moved on the sheet: C3, C4, C9, D2, D3, D6, IC2, IC3, J5, J6, K1, L1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

Commit message: Completes most PCB routing
Parts:
- removed C15: 10uF, easyeda2kicad:C0805, symbol Device:C
- removed C16, C19: 0.1uF, easyeda2kicad:C0402, symbol Device:C
- removed GPIO20: ~, TestPoint:TestPoint_Pad_2.0x2.0mm, symbol Connector:TestPoint
- removed IC3: ADC088S022CIMTX_NOPB, easyeda2kicad:TSSOP-16_L5.0-W4.4-P0.65-LS6.4-BL, symbol Drip:ADC088S022CIMTX_NOPB
- removed J6: Conn_01x03_Socket, easyeda2kicad:CONN-TH_3P-P2.50_A2501WV2-3P, symbol Connector:Conn_01x03_Socket
- removed TP10, TP5, TP6, TP7: TestPoint, TestPoint:TestPoint_Pad_2.0x2.0mm, symbol Connector:TestPoint
- added GPIO0, GPIO8: ~, TestPoint:TestPoint_Pad_2.0x2.0mm, symbol Connector:TestPoint
- added R14, R15, R16: 10000, easyeda2kicad:R1206, symbol Device:R
- added U1: ADS1115IRUGT, easyeda2kicad:X2QFN-10_L2.0-W1.5-P0.50-TL_RUG0010B, symbol Drip:ADS1115IRUGT
- R5: value 220 -> 120; footprint easyeda2kicad:RES-TH_BD2.3-L6.5-P10.50-D0.5 -> easyeda2kicad:RES-TH_BD2.2-L6.5-P10.50-D0.6; LCSC Part C714546 -> C172969
Connections:
- net +3V3 is gone; now on net +3.3V: C7.2, C8.2, IC1.1 (3V3), J7.3 (Pin_3), R1.1, R2.1
- net ACD Chip Select is gone; now on net SDA: IC1.15 (IO3)
- net IO20 is gone; now on net Flow Sensor Enable: IC1.11 (IO20/RXD), J7.5 (Pin_5)
- net +3.3V: now also R14.2, R15.2, R16.2, U1.8 (VDD)
- net Flow Sensor Enable: no longer IC1.7 (IO8)
- net GND: now also U1.1 (ADDR), U1.3 (GND)
- net IO21: now also GPIO21.1
- net SCLK: now also IC1.16 (IO2), R15.1, U1.10 (SCL); no longer IC1.17 (IO1)
- net SDA: now also R14.1, U1.9 (SDA); no longer IC1.16 (IO2)
- net ACD Program: no longer names the net of IC1.18 (IO0)
- net ACD Program: now also GPIO0.1
- net Pressure Sensor (Current) renamed Pressure Sensor Voltage
- net Pressure Sensor Voltage: now also U1.4 (AIN0)
- new net: GPIO8.1, IC1.7 (IO8)
- new net ADC Alert: IC1.17 (IO1), R16.1, U1.2 (ALERT/RDY)
- no-connect marks 7 -> 10
Other:
- moved on the sheet: C17, C18, C20, J5, R13, R5, TP9

Commit message: Polishes PCB
Other:
- moved on the sheet: C1, C10, C11, C12, C13, C14, C17, C18, C2, C20, C21, C22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
